File: diagramas/iv_diagrams/_saved__saved_iv_diagrams.sch (KiCad schematic (older format))
At the start: 15 parts

Commit message: ALU
Signed-off-by: Ricardo Mena C <rgacort12@gmail.com>
Parts:
- added U? (x5): 74AUC2G86, symbol 74xGxx:74AUC2G86
Connections:
- wire segments 62 -> 93
