File: diagramas/iv_diagrams/_saved_iv_diagrams.sch (KiCad schematic (older format))
At the start: 14 parts

Commit message: ALU
Signed-off-by: Ricardo Mena C <rgacort12@gmail.com>
Parts:
- removed U? (x2): 74AHC1G08, symbol 74xGxx:74AHC1G08
- added U?: 74AHC1G08, symbol 74xGxx:74AHC1G08
- added U? (x5): 74AUC2G86, symbol 74xGxx:74AUC2G86
- added U?: 74AUC2G32, symbol 74xGxx:74AUC2G32
- added U?: 74AHC1G86, symbol 74xGxx:74AHC1G86
Connections:
- net labels added: A_0, A_1, A_2, A_3, B_0, B_1, B_2, B_3, C_0, C_1, C_2, C_3, Vector_Cout
- net labels removed: &a, 0001, 01, 1111, Cout
- wire segments 29 -> 93
